File: Electronics/PCB/ESE_RuizHerbelinAsfary/Power_Supply.kicad_sch (KiCad schematic)
At the start: 0 parts

Commit message: added test pin
Parts:
- added C401: 10uF, symbol Device:C_Small
- added C402: 22uF, symbol Device:C_Small
- added C403, C404: 1uF, symbol Device:C_Small
- added J401: Conn_01x02_Male, symbol Connector:Conn_01x02_Male
- added S401: 1A11-NF5STSE-B, 1A11-NF5STSE-B, symbol SamacSys_Parts:1A11-NF5STSE-B
- added U401: AZ1117_Reg5V, symbol AZ1117_Reg5V:AZ1117_Reg5V
- added U402: MIC5317_Reg3V, symbol MIC5317_Reg3V:MIC5317_Reg3V
Connections:
- new net: J401.1 (Pin_1), S401.1
- new net +3.3V: C404.1, U402.3 (OUTPUT)
- new net +5V: C402.1, C403.1, U401.2 (VOUT_OUTPUT), U402.0 (VIN), U402.1 (EN)
- new net +BATT: C401.1, S401.2, U401.0 (VIN_INPUT)
- new net GND: C401.2, C402.2, C403.2, C404.2, J401.2 (Pin_2), U401.1 (GND), U402.2 (GND)
Other:
- note added: "Bloc Alimentation"
- note added: "Capteur TOF"
- note added: "Capteur infra Capteurs couleurs"
- note added: "Servomoteur + Drivers moteurs"

Commit message: PCB finished
Connections:
- no-connect marks 0 -> 1
Changed lines of the file:
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@@
   (junction (at 82.55 68.58) (diameter 0) (color 0 0 0 0)
   )
+  (no_connect (at 60.96 71.12))
   (wire (pts (xy 130.81 68.58) (xy 130.81 73.66))
     (stroke (width 0) (type default) (color 0 0 0 0))
