File: Electronics/PCB/ESE_RuizHerbelinAsfary/STM32.kicad_sch (KiCad schematic)
At the start: 0 parts

Commit message: added test pin
Parts:
- added C301: 1uF, symbol Device:C_Small
- added C302: 4.7uF, symbol Device:C_Small
- added C303, C304: 100nF, symbol Device:C_Small
- added C305: 1 uF, symbol Device:C_Small
- added C306, C307: C_Small, Capacitor_SMD:C_0603_1608Metric_Pad1.08x0.95mm_HandSolder, symbol Device:C_Small
- added D301: Green, LED_SMD:LED_0603_1608Metric_Pad1.05x0.95mm_HandSolder, symbol Device:LED_Small
- added D302: Blue, LED_SMD:LED_0603_1608Metric_Pad1.05x0.95mm_HandSolder, symbol Device:LED_Small
- added D303: Red, LED_SMD:LED_0603_1608Metric_Pad1.05x0.95mm_HandSolder, symbol Device:LED_Small
- added J301: Conn_02x07_Odd_Even, Connector_PinHeader_1.27mm:PinHeader_2x07_P1.27mm_Vertical_SMD, symbol Connector_Generic:Conn_02x07_Odd_Even
- added JP301, JP302: SolderJumper_2_Open, symbol Jumper:SolderJumper_2_Open
- added JP303, JP304: SolderJumper_2_Open, Jumper:SolderJumper-2_P1.3mm_Open_TrianglePad1.0x1.5mm, symbol Jumper:SolderJumper_2_Open
- added L301: 600R@100MHz, symbol Device:L_Small
- added R301: 100k, Resistor_SMD:R_0603_1608Metric_Pad0.98x0.95mm_HandSolder, symbol Device:R_Small
- added R302, R303: R_Small, Resistor_SMD:R_0603_1608Metric_Pad0.98x0.95mm_HandSolder, symbol Device:R_Small
- added R304, R305, R307, R308: 1k, Resistor_SMD:R_0603_1608Metric_Pad0.98x0.95mm_HandSolder, symbol Device:R_Small
- added R306: 1.2k, Resistor_SMD:R_0603_1608Metric_Pad0.98x0.95mm_HandSolder, symbol Device:R_Small
- added U301: STM32G070RBTx, symbol STM32G070RBTx:STM32G070RBTx
- added Y301: 16MHz, Crystal:Crystal_SMD_EuroQuartz_MT-4Pin_3.2x2.5mm, symbol Device:Crystal_GND24_Small
Connections:
- new net: D303.1 (K), R308.1
- new net: C307.1, R303.1, Y301.2
- new net: R303.2, U301.11 (PF1-OSC_OUT)
- new net: C306.1, U301.10 (PF0-OSC_IN), Y301.4
- new net: D301.1 (K), R305.1
- new net: JP301.1 (A), R301.2
- new net: JP302.1 (A), R302.2
- new net: J301.13 (Pin_13), JP303.2 (B)
- new net: D302.1 (K), R307.1
- new net: J301.14 (Pin_14), JP304.2 (B)
- new net +3.3V: D301.2 (A), J301.3 (Pin_3), R301.1, U301.6 (VBAT), U301.7 (VREF+)
- new net +5V: D302.2 (A)
- new net +BATT: R304.1
- new net GND: C301.2, C302.2, C303.2, C304.2, C305.2, C306.2, C307.2, J301.11 (Pin_11), J301.5 (Pin_5), J301.7 (Pin_7), R302.1, R305.2, R306.2, R307.2, R308.2, U301.9 (VSS/VSSA), Y301.1, Y301.3
- new net NRST: C305.1, J301.12 (Pin_12), U301.12 (NRST)
- new net PA0: U301.17 (PA0)
- new net PA1: U301.18 (PA1)
- new net PA10: U301.42 (PA10)
- new net PA11: U301.43 (PA11[PA9])
- new net PA12: U301.44 (PA12[PA10])
- new net PA15: U301.47 (PA15)
- new net PA4: U301.21 (PA4)
- new net PA5: U301.22 (PA5)
- new net PA6: U301.23 (PA6)
- new net PA7: U301.24 (PA7)
- new net PA8: U301.36 (PA8)
- new net PA9: U301.37 (PA9)
- new net PB0: U301.27 (PB0)
- new net PB1: U301.28 (PB1)
- new net PB10: U301.30 (PB10)
- new net PB11: U301.31 (PB11)
- new net PB12: U301.32 (PB12)
- new net PB13: U301.33 (PB13)
- new net PB14: U301.34 (PB14)
- new net PB15: U301.35 (PB15)
- new net PB2: U301.29 (PB2)
- new net PB3: U301.57 (PB3)
- new net PB4: U301.58 (PB4)
- new net PB5: U301.59 (PB5)
- new net PB6: U301.60 (PB6)
- new net PB7: U301.61 (PB7)
- new net PB8: U301.62 (PB8)
- new net PB9: U301.63 (PB9)
- new net PC0: U301.13 (PC0)
- new net PC1: U301.14 (PC1)
- new net PC10: U301.64 (PC10)
- new net PC11: U301.1 (PC11)
- new net PC12: U301.2 (PC12)
- new net PC13: U301.3 (PC13)
- new net PC2: U301.15 (PC2)
- new net PC3: U301.16 (PC3)
- new net PC4: U301.25 (PC4)
- new net PC5: U301.26 (PC5)
- new net PC6: U301.38 (PC6)
- new net PC7: U301.39 (PC7)
- new net PC8: U301.48 (PC8)
- new net PC9: U301.49 (PC9)
- new net PD0: U301.50 (PD0)
- new net PD1: U301.51 (PD1)
- new net PD2: U301.52 (PD2)
- new net PD3: U301.53 (PD3)
- new net PD4: U301.54 (PD4)
- new net PD5: U301.55 (PD5)
- new net PD6: U301.56 (PD6)
- new net PD8: U301.40 (PD8)
- new net PD9: U301.41 (PD9)
- new net POWER_STATUS_ADC: R304.2, R306.1, U301.4 (PC14-OSC32_IN)
- new net POWER_STATUS_LED: D303.2 (A), U301.5 (PC15-OSC32_OUT)
- new net SWCLK: J301.6 (Pin_6), JP302.2 (B), U301.46 (PA14-BOOT0)
- new net SWDIO: J301.4 (Pin_4), JP301.2 (B), U301.45 (PA13)
- new net VCP_RX: JP303.1 (A), U301.20 (PA3)
- new net VCP_TX: JP304.1 (A), U301.19 (PA2)
- new net VDD: C301.1, C302.1, C303.1, L301.2
- new net VDDA: C304.1, L301.1, U301.8 (VDD/VDDA)
- no-connect marks 0 -> 5
Other:
- note added: "BYPASS Capacitor"
- note added: "Power LED"
- note added: "STM32F070"
- note added: "Serial Wire Debug"
- note added: "The Bypass capacitor must be placed near the corresponding power input"
- note added: "close to VBAT"
- note added: "close to VDD"
- note added: "close to VREF"

Commit message: PCB finished
Connections:
- net PA0 is gone; now on net POWER_STATUS_ADC: U301.17 (PA0)
- net PC3 is gone; now on net POWER_STATUS_LED: U301.16 (PC3)
- net POWER_STATUS_ADC: no longer U301.4 (PC14-OSC32_IN)
- net POWER_STATUS_LED: no longer U301.5 (PC15-OSC32_OUT)
- new net PC14: U301.4 (PC14-OSC32_IN)
- new net PC15: U301.5 (PC15-OSC32_OUT)
Changed lines of the file:
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@@
-    (effects (font (size 1.27 1.27)) (justify right bottom))
-  )
-  (label "POWER_STATUS_ADC" (at 140.97 69.85 180)
     (effects (font (size 1.27 1.27)) (justify right bottom))
   )
@@
     (effects (font (size 1.27 1.27)) (justify left bottom))
   )
-  (label "POWER_STATUS_LED" (at 140.97 72.39 180)
+  (label "VCP_TX" (at 71.12 39.37 180)
     (effects (font (size 1.27 1.27)) (justify right bottom))
   )
-  (label "VCP_TX" (at 71.12 39.37 180)
+  (label "POWER_STATUS_LED" (at 140.97 41.91 180)
+    (effects (font (size 1.27 1.27)) (justify right bottom))
+  )
+  (label "POWER_STATUS_ADC" (at 71.12 34.29 180)
     (effects (font (size 1.27 1.27)) (justify right bottom))
   )
@@
     (effects (font (size 1.27 1.27)) (justify left))
   )
+  (hierarchical_label "PC14" (shape input) (at 140.97 69.85 180)
+    (effects (font (size 1.27 1.27)) (justify right))
+  )
   (hierarchical_label "PB8" (shape input) (at 105.41 54.61 0)
     (effects (font (size 1.27 1.27)) (justify left))
@@
     (effects (font (size 1.27 1.27)) (justify left))
   )
-  (hierarchical_label "PA11" (shape input) (at 71.12 62.23 180)
+  (hierarchical_label "PC15" (shape input) (at 140.97 72.39 180)
     (effects (font (size 1.27 1.27)) (justify right))
   )
-  (hierarchical_label "PC3" (shape input) (at 140.97 41.91 180)
+  (hierarchical_label "PA11" (shape input) (at 71.12 62.23 180)
     (effects (font (size 1.27 1.27)) (justify right))
   )
@@
     (effects (font (size 1.27 1.27)) (justify right))
   )
-  (hierarchical_label "PA0" (shape input) (at 71.12 34.29 180)
-    (effects (font (size 1.27 1.27)) (justify right))
-  )
