File: Electronics/ESE_RuizHerbelinAsfary/Actuator.kicad_sch (KiCad schematic)
At the start: 20 parts, among them J501 Conn_01x06_Female, J502 Conn_01x06_Female, J503 Conn_01x03_Female, U501 ZXBM5210-S, U502 ZXBM5210-S

Commit message: Add files via upload
Connections:
- net MotorLFT_P: now also J501.6 (Pin_6), JP506.2 (B)
Changed lines of the file:
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@@
     (effects (font (size 1.27 1.27)) (justify left bottom))
   )
-  (label "MotorLFT_P_JP" (at 91.44 93.98 0)
+  (label "MotorLFT_P_JP" (at 92.71 93.98 0)
     (effects (font (size 1.27 1.27)) (justify left bottom))
   )
@@
     (effects (font (size 1.27 1.27)) (justify left bottom))
   )
-  (label "MotorLFT_P" (at 107.95 96.52 0)
+  (label "MotorLFT_P" (at 107.95 93.98 0)
     (effects (font (size 1.27 1.27)) (justify left bottom))
   )
