File: Electronics/ESE_RuizHerbelinAsfary/ESE_RuizHerbelinAsfary.kicad_pcb (KiCad board)
At the start: 4 copper layers, 112 x 52 mm, 77 parts, among them J101 I2C1, J102 MTRX_test, J103 UART3, J104 I2C1, J105 MTRX_test, J201 Conn_01x07_Female, J202 Conn_01x07_Female, J203 Conn_01x03_Female, J204 Conn_01x03_Female, J205 Conn_01x05_Female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

Commit message: Add files via upload
Parts:
- removed R203, R206: 10k, Resistor_SMD:R_0603_1608Metric_Pad0.98x0.95mm_HandSolder
- added JP201: SolderJumper_2_Open, Jumper:SolderJumper-2_P1.3mm_Open_TrianglePad1.0x1.5mm, F.Cu at (62.0, 34.0)
- added JP202: SolderJumper_2_Open, Jumper:SolderJumper-2_P1.3mm_Open_TrianglePad1.0x1.5mm, F.Cu at (62.0, 36.7)
- moved C305 37.7 mm to (100.4, 47.5), turned to 90 degrees
- moved JP304 15.3 mm to (91.9, 46.0), turned to 0 degrees
- moved JP303 12.6 mm to (99.0, 35.0), turned to 90 degrees
- moved J301 5.68 mm to (92.6, 38.1), turned to 180 degrees
- moved C306 5.13 mm to (67.2, 41.7), turned to 180 degrees
- moved JP504 4.78 mm to (107.1, 30.8), turned to 0 degrees
- moved C303 3.37 mm to (67.3, 36.5)
- moved SW301 2.22 mm to (106.6, 46.2)
- moved C304 1.86 mm to (67.2, 40.1)
- moved C302 1.54 mm to (67.3, 34.8)
- moved L301 1.46 mm to (67.0, 38.3)
- moved C501 1.36 mm to (41.5, 27.6)
- moved JP502 0.95 mm to (41.5, 29.8)
- moved U402 0.78 mm to (49.1, 24.8)
- moved C404 0.56 mm to (49.1, 27.9)
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Connections:
- net Net-(J501-Pad6) renamed /Actuator/MotorLFT_P
- J201 pad 2: unconnected-(J201-Pad2) -> +3.3V
- J201 pad 6: Net-(J201-Pad6) -> +3.3V
- J201 pad 7: unconnected-(J201-Pad7) -> /Sensor/GPIO_TOF_1_JP
- J202 pad 2: unconnected-(J202-Pad2) -> +3.3V
- J202 pad 6: Net-(J202-Pad6) -> +3.3V
- J202 pad 7: unconnected-(J202-Pad7) -> /Sensor/GPIO_TOF_2_JP
- J205 pad 4: unconnected-(J205-Pad4) -> /STM32/LED1
- J207 pad 4: unconnected-(J207-Pad4) -> /STM32/LED2
- J401 pad 1: /Power_Supply/Alim -> GND
- J401 pad 2: GND -> /Power_Supply/Alim
- U301 pad 3: /STM32/PC13 -> /Sensor/GPIO_TOF_1
- U301 pad 33: /STM32/PB13 -> /STM32/LED1
- U301 pad 34: /STM32/PB14 -> /STM32/LED2
- U301 pad 4: /STM32/PC14 -> /Sensor/GPIO_TOF_2
- U301 pad 51: /Actuator/FWD_RightMotor_PWM -> /Actuator/REV_RightMotor_PWM
- U301 pad 61: /Actuator/REV_RightMotor_PWM -> /Actuator/FWD_RightMotor_PWM
Routing:
- net +5V: track 312.6 -> 60.0 mm, vias 2 -> 4
- net +3.3V: track 43.9 -> 121.7 mm
- net /Actuator/UART_Servomoteur: track 100.1 -> 35.0 mm, vias 6 -> 2
- net /STM32/NRST: track 98.0 -> 51.6 mm, vias 8 -> 3
- net /Sensor/GPIO_TOF_1_JP: track 0.00 -> 34.5 mm, vias 0 -> 2
- net /STM32/LED2: track 0.00 -> 31.3 mm, vias 0 -> 1
- net Net-(J201-Pad6): track 28.2 -> 0.00 mm, vias 2 -> 0
- net /STM32/LED1: track 0.00 -> 27.9 mm, vias 0 -> 1
- net /STM32/VCP_TX: track 47.1 -> 20.8 mm
- net /Sensor/GPIO_TOF_2_JP: track 0.00 -> 20.1 mm, vias 0 -> 1
- net /Actuator/EncoderB_Right: track 45.4 -> 63.8 mm, vias 1 -> 2
- net /Actuator/EncoderA_Right: track 40.4 -> 57.4 mm
- net /STM32/VCP_TX_JP: track 3.60 -> 20.5 mm, vias 0 -> 2
- net /Sensor/GPIO_TOF_2: track 0.00 -> 16.6 mm
- net /Sensor/GPIO_TOF_1: track 0.00 -> 15.3 mm
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- added copper zone on In2.Cu, net +5V
Other:
- board text added: "+"
- board text added: "-"
