File: Electronics/ESE_RuizHerbelinAsfary/ESE_RuizHerbelinAsfary.kicad_sch (KiCad schematic)
At the start: 9 parts, among them J101 I2C1, J102 MTRX_test, J103 UART3, J104 I2C1, J105 MTRX_test

Commit message: Add files via upload
Connections:
- no-connect marks 31 -> 25
Other:
- sheet STM32 ports: added GPIO_TOF_1, GPIO_TOF_2, LED1, LED2; removed PB13, PB14, PC13, PC14
- sheet Sensor ports: added GPIO_TOF_1, GPIO_TOF_2, LED1, LED2; removed none
Changed lines of the file:
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@@
   (no_connect (at 229.87 24.13))
   (no_connect (at 266.7 53.34))
-  (no_connect (at 266.7 40.64))
   (no_connect (at 194.31 24.13))
   (no_connect (at 250.19 24.13))
@@
   (no_connect (at 232.41 24.13))
   (no_connect (at 201.93 24.13))
-  (no_connect (at 266.7 68.58))
   (no_connect (at 266.7 66.04))
   (no_connect (at 189.23 24.13))
@@
   (no_connect (at 199.39 24.13))
   (no_connect (at 266.7 73.66))
-  (no_connect (at 266.7 71.12))
   (no_connect (at 245.11 24.13))
-  (no_connect (at 266.7 45.72))
   (no_connect (at 204.47 24.13))
-  (no_connect (at 266.7 43.18))
-  (no_connect (at 266.7 48.26))
   (no_connect (at 209.55 24.13))
   (no_connect (at 222.25 24.13))
@@
     (stroke (width 0) (type default) (color 0 0 0 0))
   )
+  (wire (pts (xy 158.75 60.96) (xy 177.8 60.96))
+    (stroke (width 0) (type default) (color 0 0 0 0))
+  )
   (wire (pts (xy 43.18 80.01) (xy 43.18 78.74))
     (stroke (width 0) (type default) (color 0 0 0 0))
@@
     (stroke (width 0) (type default) (color 0 0 0 0))
   )
-  (wire (pts (xy 158.75 66.04) (xy 177.8 66.04))
+  (wire (pts (xy 158.75 69.85) (xy 177.8 69.85))
     (stroke (width 0) (type default) (color 0 0 0 0))
   )
@@
     (stroke (width 0) (type default) (color 0 0 0 0))
   )
+  (wire (pts (xy 158.75 45.72) (xy 177.8 45.72))
+    (stroke (width 0) (type default) (color 0 0 0 0))
+  )
   (polyline (pts (xy 12.7 142.24) (xy 74.93 142.24))
     (stroke (width 0) (type default) (color 0 0 0 0))
@@
     (stroke (width 0) (type default) (color 0 0 0 0))
   )
+  (wire (pts (xy 158.75 48.26) (xy 177.8 48.26))
+    (stroke (width 0) (type default) (color 0 0 0 0))
+  )
   (wire (pts (xy 33.02 53.34) (xy 44.45 53.34))
     (stroke (width 0) (type default) (color 0 0 0 0))
@@
     (stroke (width 0) (type default) (color 0 0 0 0))
   )
+  (wire (pts (xy 158.75 63.5) (xy 177.8 63.5))
+    (stroke (width 0) (type default) (color 0 0 0 0))
+  )
   (wire (pts (xy 34.29 118.11) (xy 43.18 118.11))
     (stroke (width 0) (type default) (color 0 0 0 0))
@@
     (stroke (width 0) (type default) (color 0 0 0 0))
   )
-  (wire (pts (xy 158.75 63.5) (xy 177.8 63.5))
+  (wire (pts (xy 158.75 67.31) (xy 177.8 67.31))
     (stroke (width 0) (type default) (color 0 0 0 0))
   )
@@
     (effects (font (size 2.54 2.54)) (justify left bottom))
   )
-  (label "UART_Rx" (at 177.8 74.93 180)
+  (label "UART_Rx" (at 177.8 76.2 180)
     (effects (font (size 1.27 1.27)) (justify right bottom))
   )
@@
     (effects (font (size 1.27 1.27)) (justify left bottom))
   )
-  (label "UART_Tx" (at 177.8 72.39 180)
+  (label "UART_Tx" (at 177.8 73.66 180)
     (effects (font (size 1.27 1.27)) (justify right bottom))
   )
@@
       (effects (font (size 1.27 1.27)) (justify right))
     )
-    (pin "Vout2" output (at 158.75 66.04 0)
-      (effects (font (size 1.27 1.27)) (justify right))
-    )
-    (pin "Vout1" output (at 158.75 63.5 0)
+    (pin "Vout2" output (at 158.75 69.85 0)
+      (effects (font (size 1.27 1.27)) (justify right))
+    )
+    (pin "Vout1" output (at 158.75 67.31 0)
       (effects (font (size 1.27 1.27)) (justify right))
     )
@@
     )
     (pin "SCL1" output (at 158.75 58.42 0)
+      (effects (font (size 1.27 1.27)) (justify right))
+    )
+    (pin "GPIO_TOF_2" input (at 158.75 63.5 0)
+      (effects (font (size 1.27 1.27)) (justify right))
+    )
+    (pin "LED1" input (at 158.75 45.72 0)
+      (effects (font (size 1.27 1.27)) (justify right))
+    )
+    (pin "GPIO_TOF_1" input (at 158.75 60.96 0)
+      (effects (font (size 1.27 1.27)) (justify right))
+    )
+    (pin "LED2" input (at 158.75 48.26 0)
       (effects (font (size 1.27 1.27)) (justify right))
     )
@@
       (effects (font (size 1.27 1.27)) (justify right))
     )
-    (pin "PC13" input (at 266.7 71.12 0)
-      (effects (font (size 1.27 1.27)) (justify right))
-    )
     (pin "PC12" input (at 266.7 73.66 0)
       (effects (font (size 1.27 1.27)) (justify right))
@@
       (effects (font (size 1.27 1.27)) (justify right))
     )
-    (pin "PB13" input (at 266.7 45.72 0)
-      (effects (font (size 1.27 1.27)) (justify right))
-    )
-    (pin "PB14" input (at 266.7 48.26 0)
-      (effects (font (size 1.27 1.27)) (justify right))
-    )
     (pin "PB12" input (at 266.7 50.8 0)
       (effects (font (size 1.27 1.27)) (justify right))
@@
       (effects (font (size 1.27 1.27)) (justify right))
     )
-    (pin "PC14" input (at 266.7 68.58 0)
-      (effects (font (size 1.27 1.27)) (justify right))
-    )
     (pin "PC15" input (at 266.7 66.04 0)
       (effects (font (size 1.27 1.27)) (justify right))
@@
       (effects (font (size 1.27 1.27)) (justify left))
     )
-    (pin "Vout2" input (at 177.8 66.04 180)
-      (effects (font (size 1.27 1.27)) (justify left))
-    )
-    (pin "Vout1" input (at 177.8 63.5 180)
-      (effects (font (size 1.27 1.27)) (justify left))
-    )
-    (pin "UART_Tx" input (at 177.8 72.39 180)
-      (effects (font (size 1.27 1.27)) (justify left))
-    )
-    (pin "UART_Rx" input (at 177.8 74.93 180)
+    (pin "Vout2" input (at 177.8 69.85 180)
+      (effects (font (size 1.27 1.27)) (justify left))
+    )
+    (pin "Vout1" input (at 177.8 67.31 180)
+      (effects (font (size 1.27 1.27)) (justify left))
+    )
+    (pin "UART_Tx" input (at 177.8 73.66 180)
+      (effects (font (size 1.27 1.27)) (justify left))
+    )
+    (pin "UART_Rx" input (at 177.8 76.2 180)
       (effects (font (size 1.27 1.27)) (justify left))
     )
@@
     )
     (pin "UART_Servomoteur" input (at 250.19 80.01 270)
+      (effects (font (size 1.27 1.27)) (justify left))
+    )
+    (pin "LED1" input (at 177.8 45.72 180)
+      (effects (font (size 1.27 1.27)) (justify left))
+    )
+    (pin "LED2" input (at 177.8 48.26 180)
+      (effects (font (size 1.27 1.27)) (justify left))
+    )
+    (pin "GPIO_TOF_1" input (at 177.8 60.96 180)
+      (effects (font (size 1.27 1.27)) (justify left))
+    )
+    (pin "GPIO_TOF_2" input (at 177.8 63.5 180)
       (effects (font (size 1.27 1.27)) (justify left))
     )
@@
       (reference "J503") (unit 1) (value "Conn_01x03_Female") (footprint "Connector_JST:JST_XH_B3B-XH-A_1x03_P2.50mm_Vertical")
     )
+    (path "/2924da36-dbac-4d9a-b64c-88077c1fc53b/ade0a2d1-7151-4e38-97da-b3062265cd63"
+      (reference "JP201") (unit 1) (value "SolderJumper_2_Open") (footprint "Jumper:SolderJumper-2_P1.3mm_Open_TrianglePad1.0x1.5mm")
+    )
+    (path "/2924da36-dbac-4d9a-b64c-88077c1fc53b/6a5271f7-01bc-41f8-937d-f890f023f727"
+      (reference "JP202") (unit 1) (value "SolderJumper_2_Open") (footprint "Jumper:SolderJumper-2_P1.3mm_Open_TrianglePad1.0x1.5mm")
+    )
     (path "/6b2f643a-955a-47ef-920e-70e4f09a6662/c8e295a3-d358-441b-8802-aa08c068fbda"
       (reference "JP303") (unit 1) (value "SolderJumper_2_Open") (footprint "Jumper:SolderJumper-2_P1.3mm_Open_TrianglePad1.0x1.5mm")
@@
       (reference "R202") (unit 1) (value "2k") (footprint "Resistor_SMD:R_0603_1608Metric_Pad0.98x0.95mm_HandSolder")
     )
-    (path "/2924da36-dbac-4d9a-b64c-88077c1fc53b/0a291567-5538-4808-a61d-150f1d396a11"
-      (reference "R203") (unit 1) (value "10k") (footprint "Resistor_SMD:R_0603_1608Metric_Pad0.98x0.95mm_HandSolder")
-    )
     (path "/2924da36-dbac-4d9a-b64c-88077c1fc53b/b5b514ad-0373-4023-9e6b-0ed86dcf4ee6"
       (reference "R204") (unit 1) (value "2k") (footprint "Resistor_SMD:R_0603_1608Metric_Pad0.98x0.95mm_HandSolder")
@@
       (reference "R205") (unit 1) (value "2k") (footprint "Resistor_SMD:R_0603_1608Metric_Pad0.98x0.95mm_HandSolder")
     )
-    (path "/2924da36-dbac-4d9a-b64c-88077c1fc53b/599cd3f9-d424-465e-b0ff-1dea85ee5064"
-      (reference "R206") (unit 1) (value "10k") (footprint "Resistor_SMD:R_0603_1608Metric_Pad0.98x0.95mm_HandSolder")
-    )
     (path "/6b2f643a-955a-47ef-920e-70e4f09a6662/171544b6-d5c0-4b3f-a7a6-d28dde489c6f"
