File: Electronics/ESE_RuizHerbelinAsfary/Power_Supply.kicad_sch (KiCad schematic)
At the start: 8 parts, among them J401 Conn_01x02_Female, U401 AZ1117_Reg5V, U402 MIC5317_Reg3V

Commit message: Add files via upload
Connections:
- net Alim: now also J401.2 (Pin_2); no longer J401.1 (Pin_1)
- net GND: now also J401.1 (Pin_1); no longer J401.2 (Pin_2)
Other:
- moved on the sheet: J401
Changed lines of the file:
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@@
+    (stroke (width 0) (type default) (color 0 0 0 0))
+  )
+  (wire (pts (xy 35.56 68.58) (xy 55.88 68.58))
     (stroke (width 0) (type default) (color 0 0 0 0))
   )
@@
     (stroke (width 0) (type default) (color 0 0 0 0))
   )
-  (wire (pts (xy 35.56 68.58) (xy 55.88 68.58))
-    (stroke (width 0) (type default) (color 0 0 0 0))
-  )
   (wire (pts (xy 204.47 68.58) (xy 204.47 73.66))
     (stroke (width 0) (type default) (color 0 0 0 0))
@@
     (stroke (width 0) (type default) (color 0 0 0 0))
   )
-  (wire (pts (xy 35.56 71.12) (xy 35.56 96.52))
-    (stroke (width 0) (type default) (color 0 0 0 0))
-  )
   (wire (pts (xy 204.47 78.74) (xy 204.47 91.44))
     (stroke (width 0) (type default) (color 0 0 0 0))
   )
   (wire (pts (xy 111.76 81.28) (xy 111.76 82.55))
+    (stroke (width 0) (type default) (color 0 0 0 0))
+  )
+  (wire (pts (xy 35.56 71.12) (xy 35.56 74.93))
     (stroke (width 0) (type default) (color 0 0 0 0))
   )
@@
     (pin "2")
   )
-  (symbol (lib_id "power:GND") (at 35.56 96.52 0) (unit 1)
-    (in_bom yes) (on_board yes) (fields_autoplaced)
-    (property "Reference" "#PWR0401" (id 0) (at 35.56 102.87 0)
-      (effects (font (size 1.27 1.27)) hide)
-    )
-    (property "Value" "GND" (id 1) (at 35.56 101.6 0))
-    (property "Footprint" "" (id 2) (at 35.56 96.52 0)
-      (effects (font (size 1.27 1.27)) hide)
-    )
-    (property "Datasheet" "" (id 3) (at 35.56 96.52 0)
+  (symbol (lib_id "power:GND") (at 35.56 74.93 0) (unit 1)
+    (in_bom yes) (on_board yes) (fields_autoplaced)
+    (property "Reference" "#PWR0401" (id 0) (at 35.56 81.28 0)
+      (effects (font (size 1.27 1.27)) hide)
+    )
+    (property "Value" "GND" (id 1) (at 35.56 80.01 0))
+    (property "Footprint" "" (id 2) (at 35.56 74.93 0)
+      (effects (font (size 1.27 1.27)) hide)
+    )
+    (property "Datasheet" "" (id 3) (at 35.56 74.93 0)
       (effects (font (size 1.27 1.27)) hide)
     )
@@
     (pin "1")
   )
-  (symbol (lib_id "Connector:Conn_01x02_Female") (at 30.48 68.58 0) (mirror y) (unit 1)
+  (symbol (lib_id "Connector:Conn_01x02_Female") (at 30.48 71.12 180) (unit 1)
     (in_bom yes) (on_board yes) (fields_autoplaced)
     (property "Reference" "J401" (id 0) (at 31.115 63.5 0))
     (property "Value" "Conn_01x02_Female" (id 1) (at 31.115 66.04 0))
-    (property "Footprint" "Connector_JST:JST_XH_B2B-XH-A_1x02_P2.50mm_Vertical" (id 2) (at 30.48 68.58 0)
-      (effects (font (size 1.27 1.27)) hide)
-    )
-    (property "Datasheet" "~" (id 3) (at 30.48 68.58 0)
-      (effects (font (size 1.27 1.27)) hide)
-    )
+    (property "Footprint" "Connector_JST:JST_XH_B2B-XH-A_1x02_P2.50mm_Vertical" (id 2) (at 30.48 71.12 0)
+      (effects (font (size 1.27 1.27)) hide)
+    )
+    (property "Datasheet" "~" (id 3) (at 30.48 71.12 0)
+      (effects (font (size 1.27 1.27)) hide)
+    )
