File: Electronics/ESE_RuizHerbelinAsfary/STM32.kicad_sch (KiCad schematic)
At the start: 24 parts, among them J301 Conn_02x07_Odd_Even, SW301 SW_MEC_5E, U301 STM32G070RBTx, Y301 16MHz

Commit message: Add files via upload
Connections:
- net FWD_RightMotor_PWM: now also U301.61 (PB7); no longer U301.51 (PD1)
- net REV_RightMotor_PWM: now also U301.51 (PD1); no longer U301.61 (PB7)
- net PB13 renamed LED1
- net PB14 renamed LED2
- net PC13 renamed GPIO_TOF_1
- net PC14 renamed GPIO_TOF_2
Changed lines of the file:
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@@
     (stroke (width 0) (type default) (color 0 0 0 0))
   )
-  (wire (pts (xy 116.84 138.43) (xy 116.84 137.16))
+  (wire (pts (xy 116.84 140.97) (xy 116.84 137.16))
     (stroke (width 0) (type default) (color 0 0 0 0))
   )
@@
     (effects (font (size 1.27 1.27)) (justify right bottom))
   )
-  (label "OSCILLO_IN_C" (at 233.68 53.34 0)
-    (effects (font (size 1.27 1.27)) (justify left bottom))
-  )
   (label "OSCILLO_IN" (at 215.9 53.34 0)
     (effects (font (size 1.27 1.27)) (justify left bottom))
@@
     (effects (font (size 1.27 1.27)) (justify left bottom))
   )
-  (label "OSCILLO_OUT_R_C" (at 233.68 63.5 0)
-    (effects (font (size 1.27 1.27)) (justify left bottom))
-  )
   (label "SWDIO" (at 210.82 128.27 0)
     (effects (font (size 1.27 1.27)) (justify left bottom))
@@
     (effects (font (size 1.27 1.27)) (justify left))
   )
-  (hierarchical_label "PB13" (shape input) (at 105.41 67.31 0)
-    (effects (font (size 1.27 1.27)) (justify left))
-  )
-  (hierarchical_label "PC13" (shape input) (at 140.97 67.31 180)
+  (hierarchical_label "LED1" (shape input) (at 105.41 67.31 0)
+    (effects (font (size 1.27 1.27)) (justify left))
+  )
+  (hierarchical_label "GPIO_TOF_1" (shape input) (at 140.97 67.31 180)
     (effects (font (size 1.27 1.27)) (justify right))
   )
@@
     (effects (font (size 1.27 1.27)) (justify left))
   )
-  (hierarchical_label "PC14" (shape input) (at 140.97 69.85 180)
+  (hierarchical_label "GPIO_TOF_2" (shape input) (at 140.97 69.85 180)
     (effects (font (size 1.27 1.27)) (justify right))
   )
@@
     (effects (font (size 1.27 1.27)) (justify right))
   )
-  (hierarchical_label "FWD_RightMotor_PWM" (shape input) (at 175.26 36.83 0)
+  (hierarchical_label "FWD_RightMotor_PWM" (shape input) (at 105.41 52.07 0)
     (effects (font (size 1.27 1.27)) (justify left))
   )
@@
     (effects (font (size 1.27 1.27)) (justify left))
   )
-  (hierarchical_label "PB14" (shape input) (at 105.41 69.85 0)
+  (hierarchical_label "LED2" (shape input) (at 105.41 69.85 0)
     (effects (font (size 1.27 1.27)) (justify left))
   )
@@
     (effects (font (size 1.27 1.27)) (justify left))
   )
-  (hierarchical_label "REV_RightMotor_PWM" (shape input) (at 105.41 52.07 0)
+  (hierarchical_label "REV_RightMotor_PWM" (shape input) (at 175.26 36.83 0)
     (effects (font (size 1.27 1.27)) (justify left))
   )
@@
     (pin "2")
   )
-  (symbol (lib_id "power:GND") (at 116.84 138.43 0) (unit 1)
-    (in_bom yes) (on_board yes) (fields_autoplaced)
-    (property "Reference" "#PWR0301" (id 0) (at 116.84 144.78 0)
-      (effects (font (size 1.27 1.27)) hide)
-    )
-    (property "Value" "GND" (id 1) (at 116.84 143.51 0))
-    (property "Footprint" "" (id 2) (at 116.84 138.43 0)
-      (effects (font (size 1.27 1.27)) hide)
-    )
-    (property "Datasheet" "" (id 3) (at 116.84 138.43 0)
-      (effects (font (size 1.27 1.27)) hide)
-    )
+  (symbol (lib_id "power:GND") (at 116.84 140.97 0) (unit 1)
+    (in_bom yes) (on_board yes) (fields_autoplaced)
+    (property "Reference" "#PWR0301" (id 0) (at 116.84 147.32 0)
+      (effects (font (size 1.27 1.27)) hide)
+    )
+    (property "Value" "GND" (id 1) (at 116.84 146.05 0))
+    (property "Footprint" "" (id 2) (at 116.84 140.97 0)
+      (effects (font (size 1.27 1.27)) hide)
+    )
+    (property "Datasheet" "" (id 3) (at 116.84 140.97 0)
+      (effects (font (size 1.27 1.27)) hide)
+    )
