File: Electronics/ESE_RuizHerbelinAsfary/Sensor.kicad_sch (KiCad schematic)
At the start: 14 parts, among them J201 Conn_01x07_Female, J202 Conn_01x07_Female, J203 Conn_01x03_Female, J204 Conn_01x03_Female, J205 Conn_01x05_Female, J206 Conn_01x05_Female, J207 Conn_01x05_Female, J208 Conn_01x05_Female

Commit message: Add files via upload
Parts:
- removed R203, R206: 10k, Resistor_SMD:R_0603_1608Metric_Pad0.98x0.95mm_HandSolder, symbol Device:R_Small
- added JP201, JP202: SolderJumper_2_Open, Jumper:SolderJumper-2_P1.3mm_Open_TrianglePad1.0x1.5mm, symbol Jumper:SolderJumper_2_Open
Connections:
- net +3.3V: now also J201.2 (Pin_2), J201.6 (Pin_6), J202.2 (Pin_2), J202.6 (Pin_6)
- net LED1: now reaches J205.4 (Pin_4)
- net LED2: now reaches J207.4 (Pin_4)
- net GPIO_TOF_2_JP: now reaches J202.7 (Pin_7)
- net GPIO_TOF_2_JP: now also JP202.1 (A)
- net GPIO_TOF_1_JP: now reaches J201.7 (Pin_7)
- net GPIO_TOF_1_JP: now also JP201.1 (A)
- new net GPIO_TOF_1: JP201.2 (B)
- new net GPIO_TOF_2: JP202.2 (B)
- no-connect marks 6 -> 0
Changed lines of the file:
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@@
   (junction (at 63.5 62.23) (diameter 0) (color 0 0 0 0)
   )
-  (no_connect (at 91.44 55.88))
-  (no_connect (at 50.8 54.61))
-  (no_connect (at 50.8 67.31))
-  (no_connect (at 57.15 152.4))
-  (no_connect (at 204.47 139.7))
-  (no_connect (at 91.44 68.58))
+  (junction (at 93.98 53.34) (diameter 0) (color 0 0 0 0)
+  )
+  (junction (at 52.07 52.07) (diameter 0) (color 0 0 0 0)
+  )
   (wire (pts (xy 91.44 66.04) (xy 116.84 66.04))
     (stroke (width 0) (type default) (color 0 0 0 0))
@@
     (stroke (width 0) (type default) (color 0 0 0 0))
   )
+  (wire (pts (xy 50.8 67.31) (xy 53.34 67.31))
+    (stroke (width 0) (type default) (color 0 0 0 0))
+  )
   (wire (pts (xy 63.5 52.07) (xy 63.5 53.34))
     (stroke (width 0) (type default) (color 0 0 0 0))
@@
     (stroke (width 0) (type default) (color 0 0 0 0))
   )
+  (wire (pts (xy 60.96 67.31) (xy 62.23 67.31))
+    (stroke (width 0) (type default) (color 0 0 0 0))
+  )
   (wire (pts (xy 50.8 57.15) (xy 54.61 57.15))
     (stroke (width 0) (type default) (color 0 0 0 0))
@@
     (stroke (width 0) (type default) (color 0 0 0 0))
   )
+  (wire (pts (xy 52.07 52.07) (xy 52.07 54.61))
+    (stroke (width 0) (type default) (color 0 0 0 0))
+  )
   (wire (pts (xy 101.6 59.69) (xy 101.6 60.96))
     (stroke (width 0) (type default) (color 0 0 0 0))
@@
     (stroke (width 0) (type default) (color 0 0 0 0))
   )
-  (wire (pts (xy 91.44 53.34) (xy 95.25 53.34))
+  (wire (pts (xy 50.8 54.61) (xy 52.07 54.61))
     (stroke (width 0) (type default) (color 0 0 0 0))
   )
@@
     (stroke (width 0) (type default) (color 0 0 0 0))
   )
-  (wire (pts (xy 54.61 52.07) (xy 54.61 50.8))
+  (wire (pts (xy 54.61 50.8) (xy 54.61 52.07))
     (stroke (width 0) (type default) (color 0 0 0 0))
   )
@@
     (stroke (width 0) (type default) (color 0 0 0 0))
   )
+  (wire (pts (xy 76.2 59.69) (xy 76.2 64.77))
+    (stroke (width 0) (type default) (color 0 0 0 0))
+  )
   (wire (pts (xy 226.06 142.24) (xy 228.6 142.24))
     (stroke (width 0) (type default) (color 0 0 0 0))
   )
-  (wire (pts (xy 95.25 53.34) (xy 95.25 52.07))
+  (wire (pts (xy 50.8 52.07) (xy 52.07 52.07))
+    (stroke (width 0) (type default) (color 0 0 0 0))
+  )
+  (wire (pts (xy 95.25 52.07) (xy 95.25 53.34))
     (stroke (width 0) (type default) (color 0 0 0 0))
   )
@@
     (stroke (width 0) (type default) (color 0 0 0 0))
   )
-  (wire (pts (xy 116.84 59.69) (xy 116.84 60.96))
+  (wire (pts (xy 91.44 53.34) (xy 93.98 53.34))
+    (stroke (width 0) (type default) (color 0 0 0 0))
+  )
+  (wire (pts (xy 116.84 59.69) (xy 116.84 66.04))
     (stroke (width 0) (type default) (color 0 0 0 0))
   )
@@
     (stroke (width 0) (type default) (color 0 0 0 0))
   )
+  (wire (pts (xy 52.07 52.07) (xy 54.61 52.07))
+    (stroke (width 0) (type default) (color 0 0 0 0))
+  )
   (wire (pts (xy 226.06 134.62) (xy 232.41 134.62))
     (stroke (width 0) (type default) (color 0 0 0 0))
@@
     (stroke (width 0) (type default) (color 0 0 0 0))
   )
-  (wire (pts (xy 50.8 52.07) (xy 54.61 52.07))
-    (stroke (width 0) (type default) (color 0 0 0 0))
-  )
   (wire (pts (xy 91.44 60.96) (xy 101.6 60.96))
     (stroke (width 0) (type default) (color 0 0 0 0))
@@
     (stroke (width 0) (type default) (color 0 0 0 0))
   )
+  (wire (pts (xy 91.44 55.88) (xy 93.98 55.88))
+    (stroke (width 0) (type default) (color 0 0 0 0))
+  )
   (wire (pts (xy 91.44 63.5) (xy 104.14 63.5))
     (stroke (width 0) (type default) (color 0 0 0 0))
@@
     (stroke (width 0) (type default) (color 0 0 0 0))
   )
+  (wire (pts (xy 91.44 68.58) (xy 95.25 68.58))
+    (stroke (width 0) (type default) (color 0 0 0 0))
+  )
+  (wire (pts (xy 93.98 53.34) (xy 93.98 55.88))
+    (stroke (width 0) (type default) (color 0 0 0 0))
+  )
   (wire (pts (xy 165.1 63.5) (xy 168.91 63.5))
     (stroke (width 0) (type default) (color 0 0 0 0))
   )
+  (wire (pts (xy 102.87 68.58) (xy 105.41 68.58))
+    (stroke (width 0) (type default) (color 0 0 0 0))
+  )
   (wire (pts (xy 57.15 144.78) (xy 63.5 144.78))
     (stroke (width 0) (type default) (color 0 0 0 0))
@@
   )
   (wire (pts (xy 57.15 149.86) (xy 59.69 149.86))
+    (stroke (width 0) (type default) (color 0 0 0 0))
+  )
+  (wire (pts (xy 93.98 53.34) (xy 95.25 53.34))
     (stroke (width 0) (type default) (color 0 0 0 0))
   )
@@
     (effects (font (size 2.54 2.54)) (justify left bottom))
   )
+  (label "GPIO_TOF_1" (at 60.96 67.31 0)
+    (effects (font (size 1.27 1.27)) (justify left bottom))
+  )
+  (label "GPIO_TOF_1_JP" (at 52.07 67.31 0)
+    (effects (font (size 1.27 1.27)) (justify left bottom))
+  )
+  (label "GPIO_TOF_2_JP" (at 92.71 68.58 0)
+    (effects (font (size 1.27 1.27)) (justify left bottom))
+  )
+  (label "GPIO_TOF_2" (at 104.14 68.58 0)
+    (effects (font (size 1.27 1.27)) (justify left bottom))
+  )
   (hierarchical_label "S3" (shape output) (at 228.6 139.7 0)
     (effects (font (size 1.27 1.27)) (justify left))
   )
+  (hierarchical_label "GPIO_TOF_2" (shape output) (at 105.41 68.58 0)
+    (effects (font (size 1.27 1.27)) (justify left))
+  )
   (hierarchical_label "Out" (shape output) (at 81.28 154.94 0)
     (effects (font (size 1.27 1.27)) (justify left))
   )
+  (hierarchical_label "GPIO_TOF_1" (shape output) (at 62.23 67.31 0)
+    (effects (font (size 1.27 1.27)) (justify left))
+  )
   (hierarchical_label "SCL2" (shape output) (at 106.68 63.5 0)
+    (effects (font (size 1.27 1.27)) (justify left))
+  )
+  (hierarchical_label "LED2" (shape input) (at 204.47 139.7 0)
     (effects (font (size 1.27 1.27)) (justify left))
   )
@@
   )
   (hierarchical_label "SDA2" (shape output) (at 106.68 60.96 0)
+    (effects (font (size 1.27 1.27)) (justify left))
+  )
+  (hierarchical_label "LED1" (shape input) (at 57.15 152.4 0)
     (effects (font (size 1.27 1.27)) (justify left))
   )
@@
     (pin "2")
   )
-  (symbol (lib_id "Device:R_Small") (at 76.2 62.23 180) (unit 1)
-    (in_bom yes) (on_board yes)
-    (property "Reference" "R203" (id 0) (at 73.66 63.5 90))
-    (property "Value" "10k" (id 1) (at 73.66 59.69 90))
-    (property "Footprint" "Resistor_SMD:R_0603_1608Metric_Pad0.98x0.95mm_HandSolder" (id 2) (at 76.2 62.23 0)
-      (effects (font (size 1.27 1.27)) hide)
-    )
-    (property "Datasheet" "~" (id 3) (at 76.2 62.23 0)
-      (effects (font (size 1.27 1.27)) hide)
-    )
-    (pin "1")
-    (pin "2")
-  )
   (symbol (lib_id "Connector:Conn_01x05_Female") (at 52.07 149.86 0) (mirror y) (unit 1)
     (in_bom yes) (on_board yes)
@@
     (pin "1")
   )
-  (symbol (lib_id "Device:R_Small") (at 116.84 63.5 180) (unit 1)
-    (in_bom yes) (on_board yes)
-    (property "Reference" "R206" (id 0) (at 114.3 64.77 90))
-    (property "Value" "10k" (id 1) (at 114.3 60.96 90))
-    (property "Footprint" "Resistor_SMD:R_0603_1608Metric_Pad0.98x0.95mm_HandSolder" (id 2) (at 116.84 63.5 0)
-      (effects (font (size 1.27 1.27)) hide)
-    )
-    (property "Datasheet" "~" (id 3) (at 116.84 63.5 0)
-      (effects (font (size 1.27 1.27)) hide)
-    )
-    (pin "1")
-    (pin "2")
-  )
   (symbol (lib_id "power:+5V") (at 199.39 62.23 0) (unit 1)
     (in_bom yes) (on_board yes)
@@
     )
     (pin "1")
+  )
+  (symbol (lib_id "Jumper:SolderJumper_2_Open") (at 99.06 68.58 0) (unit 1)
+    (in_bom yes) (on_board yes) (fields_autoplaced)
+    (property "Reference" "JP202" (id 0) (at 99.06 62.23 0))
+    (property "Value" "SolderJumper_2_Open" (id 1) (at 99.06 64.77 0))
+    (property "Footprint" "Jumper:SolderJumper-2_P1.3mm_Open_TrianglePad1.0x1.5mm" (id 2) (at 99.06 68.58 0)
+      (effects (font (size 1.27 1.27)) hide)
+    )
+    (property "Datasheet" "~" (id 3) (at 99.06 68.58 0)
+      (effects (font (size 1.27 1.27)) hide)
+    )
+    (pin "1")
+    (pin "2")
   )
   (symbol (lib_id "Connector:Conn_01x07_Female") (at 86.36 60.96 0) (mirror y) (unit 1)
@@
     (pin "1")
   )
+  (symbol (lib_id "Jumper:SolderJumper_2_Open") (at 57.15 67.31 0) (unit 1)
+    (in_bom yes) (on_board yes) (fields_autoplaced)
+    (property "Reference" "JP201" (id 0) (at 57.15 60.96 0))
+    (property "Value" "SolderJumper_2_Open" (id 1) (at 57.15 63.5 0))
+    (property "Footprint" "Jumper:SolderJumper-2_P1.3mm_Open_TrianglePad1.0x1.5mm" (id 2) (at 57.15 67.31 0)
+      (effects (font (size 1.27 1.27)) hide)
+    )
+    (property "Datasheet" "~" (id 3) (at 57.15 67.31 0)
+      (effects (font (size 1.27 1.27)) hide)
+    )
+    (pin "1")
+    (pin "2")
+  )
   (symbol (lib_id "Connector:Conn_01x05_Female") (at 220.98 137.16 0) (mirror y) (unit 1)
